File: Venus_Repro.kicad_pcb (KiCad board)
At the start: 2 copper layers, 175.8 x 60.5 mm, 100 parts, among them CN2 PortB, IC1 MC68000FN, IC2 LMP6323, IC3 315-5700, 315-5660, 315-5708,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, IC4 MSM54C864, IC5 Z80_QFP, IC6 uPD4364CX-15, IC7 LM809

Commit message: Add files via upload
Parts:
- added C31: 0.047u, Capacitor_SMD:C_0603_1608Metric, B.Cu at (189.4, 103.7)
- C18: value 10pF -> 20pF
- EM1, EM2, EM3, EM4, EM5, EM6, EM8: value ~ -> STX222MB
- EM7: value ~ -> STB271KB
Connections:
- C32 pad 1: unconnected-(C32-Pad1) -> /BATT_TERM-
Routing:
- added copper zone on B.Cu, net /BATT_TERM+
- added copper zone on B.Cu, net /BATT_TERM-
