File: Venus_Repro.kicad_sch (KiCad schematic)
At the start: 100 parts, among them CN2 PortB, IC1 MC68000FN, IC2 LMP6323, IC3 315-5700, 315-5660, 315-5708,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, IC4 MSM54C864, IC5 Z80_QFP, IC6 uPD4364CX-15, IC7 LM809

Commit message: Add files via upload
Parts:
- added C31: 0.047u, Capacitor_SMD:C_0603_1608Metric, symbol Device:C
Connections:
- net BATT_TERM+: now also C31.1
- net BATT_TERM-: now also C32.1
- net GND: now also C31.2
Other:
- moved on the sheet: C32
Changed lines of the file:
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@@
 	)
 	(junction
+		(at 660.4 123.19)
+		(diameter 0)
+		(color 0 0 0 0)
+	)
+	(junction
 		(at 89.154 174.498)
 		(diameter 0)
@@
 	)
 	(junction
+		(at 695.198 114.3)
+		(diameter 0)
+		(color 0 0 0 0)
+	)
+	(junction
 		(at 434.34 192.786)
 		(diameter 0)
@@
 	(wire
 		(pts
+			(xy 660.4 114.3) (xy 695.198 114.3)
+		)
+		(stroke
+			(width 0)
+			(type default)
+		)
+	)
+	(wire
+		(pts
 			(xy 89.154 174.498) (xy 89.154 177.038)
 		)
@@
 	(wire
 		(pts
+			(xy 673.1 109.22) (xy 673.1 115.57)
+		)
+		(stroke
+			(width 0)
+			(type default)
+		)
+	)
+	(wire
+		(pts
 			(xy 719.074 173.99) (xy 719.074 175.26)
 		)
@@
 	(wire
 		(pts
-			(xy 695.198 109.22) (xy 695.96 109.22)
-		)
-		(stroke
-			(width 0)
-			(type default)
-		)
-	)
-	(wire
-		(pts
 			(xy 715.772 60.96) (xy 685.8 60.96)
 		)
@@
 	(wire
 		(pts
+			(xy 660.4 114.3) (xy 660.4 115.57)
+		)
+		(stroke
+			(width 0)
+			(type default)
+		)
+	)
+	(wire
+		(pts
 			(xy 730.758 157.988) (xy 749.3 157.988)
 		)
@@
 	(wire
 		(pts
+			(xy 673.1 109.22) (xy 695.96 109.22)
+		)
+		(stroke
+			(width 0)
+			(type default)
+		)
+	)
+	(wire
+		(pts
 			(xy 307.34 108.712) (xy 304.8 108.712)
 		)
@@
 	(wire
 		(pts
+			(xy 660.4 123.19) (xy 673.1 123.19)
+		)
+		(stroke
+			(width 0)
+			(type default)
+		)
+	)
+	(wire
+		(pts
 			(xy 728.218 203.2) (xy 728.218 213.36)
 		)
@@
 	(wire
 		(pts
-			(xy 695.198 114.3) (xy 695.96 114.3)
-		)
-		(stroke
-			(width 0)
-			(type default)
-		)
-	)
-	(wire
-		(pts
 			(xy 442.214 192.786) (xy 442.214 194.056)
 		)
@@
 	(wire
 		(pts
+			(xy 695.198 114.3) (xy 695.96 114.3)
+		)
+		(stroke
+			(width 0)
+			(type default)
+		)
+	)
+	(wire
+		(pts
 			(xy 675.64 50.8) (xy 675.64 63.5)
 		)
@@
 	)
 	(label "BATT_TERM-"
-		(at 695.198 109.22 180)
+		(at 694.69 109.22 180)
 		(effects
 			(font
@@
 	)
 	(label "BATT_TERM+"
-		(at 695.198 114.3 180)
+		(at 694.69 114.3 180)
 		(effects
 			(font
@@
 	)
 	(symbol
+		(lib_id "Device:C")
+		(at 660.4 119.38 0)
+		(mirror y)
+		(unit 1)
+		(exclude_from_sim yes)
+		(in_bom no)
+		(on_board yes)
+		(dnp no)
+		(fields_autoplaced yes)
+		(property "Reference" "C31"
+			(at 656.59 118.1099 0)
+			(effects
+				(font
+					(size 1.27 1.27)
+				)
+				(justify left)
+			)
+		)
+		(property "Value" "0.047u"
+			(at 656.59 120.6499 0)
+			(effects
+				(font
+					(size 1.27 1.27)
+				)
+				(justify left)
+			)
+		)
+		(property "Footprint" "Capacitor_SMD:C_0603_1608Metric"
+			(at 659.4348 123.19 0)
+			(effects
+				(font
+					(size 1.27 1.27)
+				)
+				(hide yes)
+			)
+		)
+		(property "Datasheet" "~"
+			(at 660.4 119.38 0)
+			(effects
+				(font
+					(size 1.27 1.27)
+				)
+				(hide yes)
+			)
+		)
+		(property "Description" "Unpolarized capacitor"
+			(at 660.4 119.38 0)
+			(effects
+				(font
+					(size 1.27 1.27)
+				)
+				(hide yes)
+			)
+		)
+		(pin "1"
+		)
+		(pin "2"
+		)
+		(instances
+			(project "Venus_Repro"
+				(path "/dfd7aaab-7d44-4d59-9786-e69f1eb84d43"
+					(reference "C31")
+					(unit 1)
+				)
+			)
+		)
+	)
+	(symbol
 		(lib_id "Device:R_US")
 		(at 803.148 96.52 180)
@@
 	(symbol
 		(lib_id "Device:C")
-		(at 48.26 187.198 0)
+		(at 673.1 119.38 0)
+		(mirror y)
 		(unit 1)
 		(exclude_from_sim yes)
@@
 		(fields_autoplaced yes)
 		(property "Reference" "C32"
-			(at 52.07 185.9279 0)
+			(at 669.29 118.1099 0)
 			(effects
 				(font
@@
 		)
 		(property "Value" "C"
-			(at 52.07 188.4679 0)
+			(at 669.29 120.6499 0)
 			(effects
 				(font
@@
 		)
 		(property "Footprint" "Capacitor_SMD:C_0603_1608Metric"
-			(at 49.2252 191.008 0)
+			(at 672.1348 123.19 0)
 			(effects
 				(font
@@
 		)
 		(property "Datasheet" "~"
-			(at 48.26 187.198 0)
+			(at 673.1 119.38 0)
 			(effects
 				(font
@@
 		)
 		(property "Description" "Unpolarized capacitor"
-			(at 48.26 187.198 0)
+			(at 673.1 119.38 0)
 			(effects
 				(font
@@
 	)
 	(symbol
-		(lib_id "power:GND")
-		(at 48.26 191.008 0)
-		(unit 1)
-		(exclude_from_sim no)
-		(in_bom yes)
-		(on_board yes)
-		(dnp no)
-		(property "Reference" "#PWR047"
-			(at 48.26 197.358 0)
-			(effects
-				(font
-					(size 1.27 1.27)
-				)
-				(hide yes)
-			)
-		)
-		(property "Value" "GND"
-			(at 48.26 194.564 0)
-			(effects
-				(font
-					(size 1.27 1.27)
-				)
-			)
-		)
-		(property "Footprint" ""
-			(at 48.26 191.008 0)
-			(effects
-				(font
-					(size 1.27 1.27)
-				)
-				(hide yes)
-			)
-		)
-		(property "Datasheet" ""
-			(at 48.26 191.008 0)
-			(effects
-				(font
-					(size 1.27 1.27)
-				)
-				(hide yes)
-			)
-		)
-		(property "Description" "Power symbol creates a global label with name \"GND\" , ground"
-			(at 48.26 191.008 0)
-			(effects
-				(font
-					(size 1.27 1.27)
-				)
-				(hide yes)
-			)
-		)
-		(pin "1"
-		)
-		(instances
-			(project "Venus_Repro"
-				(path "/dfd7aaab-7d44-4d59-9786-e69f1eb84d43"
-					(reference "#PWR047")
-					(unit 1)
-				)
-			)
-		)
-	)
-	(symbol
 		(lib_id "Device:C_Polarized")
 		(at 649.732 293.37 0)
@@
 					(unit 1)
 				)
+			)
+		)
+	)
+	(symbol
+		(lib_id "power:GND")
+		(at 660.4 123.19 0)
+		(mirror y)
+		(unit 1)
+		(exclude_from_sim no)
+		(in_bom yes)
+		(on_board yes)
+		(dnp no)
+		(property "Reference" "#PWR076"
+			(at 660.4 129.54 0)
+			(effects
+				(font
+					(size 1.27 1.27)
+				)
+				(hide yes)
+			)
+		)
+		(property "Value" "GND"
+			(at 660.4 126.746 0)
+			(effects
+				(font
+					(size 1.27 1.27)
+				)
+			)
+		)
+		(property "Footprint" ""
+			(at 660.4 123.19 0)
+			(effects
+				(font
+					(size 1.27 1.27)
+				)
+				(hide yes)
+			)
+		)
+		(property "Datasheet" ""
+			(at 660.4 123.19 0)
+			(effects
+				(font
+					(size 1.27 1.27)
+				)
+				(hide yes)
+			)
+		)
+		(property "Description" "Power symbol creates a global label with name \"GND\" , ground"
+			(at 660.4 123.19 0)
+			(effects
+				(font
+					(size 1.27 1.27)
+				)
+				(hide yes)
+			)
+		)
+		(pin "1"
+		)
+		(instances
+			(project "Venus_Repro"
+				(path "/dfd7aaab-7d44-4d59-9786-e69f1eb84d43"
+					(reference "#PWR076")
+					(unit 1)
+				)
